File: tutorial-77.kicad_pcb (KiCad board)
At the start: 2 copper layers, 25 x 25 mm, 7 parts, among them J1 Conn_01x03_Pin, U1 ATtiny85-20S

Commit message: plan-b  adjust parts position
Routing:
- net Net-(J1-Pin_1): track 0.00 -> 9.88 mm
- net VCC: track 0.00 -> 7.43 mm
- net /INPUT: track 0.00 -> 5.97 mm
- net Net-(D1-A): track 0.00 -> 3.92 mm
- net Net-(D1-K): track 0.00 -> 1.94 mm
Changed lines of the file:
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@@
 		)
+	)
+	(segment
+		(start 125.715 120.955)
+		(end 123.885 120.955)
+		(width 0.1524)
+		(layer "F.Cu")
+		(net "Net-(D1-K)")
+	)
+	(segment
+		(start 123.885 120.955)
+		(end 123.81 121.03)
+		(width 0.1524)
+		(layer "F.Cu")
+		(net "Net-(D1-K)")
+	)
+	(segment
+		(start 130.16 127.46)
+		(end 129.0959 126.3959)
+		(width 0.1524)
+		(layer "F.Cu")
+		(net "VCC")
+	)
+	(segment
+		(start 129.1125 120.475)
+		(end 129.0959 120.4916)
+		(width 0.1524)
+		(layer "F.Cu")
+		(net "VCC")
+	)
+	(segment
+		(start 129.0959 120.4916)
+		(end 129.0959 122.3683)
+		(width 0.1524)
+		(layer "F.Cu")
+		(net "VCC")
+	)
+	(segment
+		(start 129.0959 126.3959)
+		(end 129.0959 122.3683)
+		(width 0.1524)
+		(layer "F.Cu")
+		(net "VCC")
+	)
+	(segment
+		(start 136.2875 119.205)
+		(end 142.145 119.205)
+		(width 0.1524)
+		(layer "F.Cu")
+		(net "/INPUT")
+	)
+	(segment
+		(start 142.145 119.205)
+		(end 142.225 119.285)
+		(width 0.1524)
+		(layer "F.Cu")
+		(net "/INPUT")
+	)
+	(segment
+		(start 126.985 117.935)
+		(end 129.1125 117.935)
+		(width 0.1524)
+		(layer "F.Cu")
+		(net "Net-(D1-A)")
+	)
+	(segment
+		(start 125.715 119.205)
+		(end 126.985 117.935)
+		(width 0.1524)
+		(layer "F.Cu")
+		(net "Net-(D1-A)")
+	)
+	(segment
+		(start 135.24 127.46)
+		(end 136.3203 127.46)
+		(width 0.1524)
+		(layer "F.Cu")
+		(net "Net-(J1-Pin_1)")
+	)
+	(segment
+		(start 136.3203 127.0147)
+		(end 142.225 121.11)
+		(width 0.1524)
+		(layer "F.Cu")
+		(net "Net-(J1-Pin_1)")
+	)
+	(segment
+		(start 136.3203 127.46)
+		(end 136.3203 127.0147)
+		(width 0.1524)
+		(layer "F.Cu")
+		(net "Net-(J1-Pin_1)")
 	)
 	(zone
